File: kicad/power_management.kicad_sch (KiCad schematic)
At the start: 30 parts, among them J17 PJ-002AH, SW1 RESET, U1 TPS54302DDCR, U12 TPS3823-33DBVR, U2 AMS1117-3.3

Commit message: fix: Resolve 5 ERC warnings — footprints, grid alignment, net conflict
1. Inductor footprint: L_4.0x4.0mm_H2.0mm → L_Taiyo-Yuden_NR-40xx
   (power_management.kicad_sch)

2. Relay footprint (×2): Relay_SPST_HF46F → Relay_SPDT_Omron_G5V-1
   (actuator_drivers.kicad_sch — K1, K2)

3. Off-grid coordinates: TPS3823 symbol and WDT_RESET label moved
   from 300.48/310.64 to 300.99/311.15 (1.27mm grid aligned)
   PWR_FLAG reference position 28.575 → 27.94
   (power_management.kicad_sch)

4. HUM_ADC/I2C_SDA overlap: Both hierarchical labels were at same
   coordinates (55.88, 107.95). Shifted I2C_SDA and downstream
   labels down by 2.54mm each to eliminate net conflict.
   (hmi_connectors.kicad_sch)

Co-Authored-By: Devin AI <158243242+devin-ai-integration[bot]@users.noreply.github.com>
Parts:
- L1: footprint Inductor_SMD:L_4.0x4.0mm_H2.0mm -> Inductor_SMD:L_Taiyo-Yuden_NR-40xx
Changed lines of the file:
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@@
     (uuid "pf-12v-001")
     (property "Reference" "#FLG01"
-      (at 25.4 28.575 0)
+      (at 25.4 27.94 0)
       (effects (font (size 1.27 1.27)) hide)
     )
@@
       (effects (font (size 1.27 1.27)))
     )
-    (property "Footprint" "Inductor_SMD:L_4.0x4.0mm_H2.0mm"
+    (property "Footprint" "Inductor_SMD:L_Taiyo-Yuden_NR-40xx"
       (at 160.02 71.12 0)
       (effects (font (size 1.27 1.27)) hide)
@@
   (symbol
     (lib_id "nebula_symbols:TPS3823-33DBVR")
-    (at 300.48 76.2 0)
+    (at 300.99 76.2 0)
     (unit 1)
     (exclude_from_sim no)
@@
     (uuid "u12-001")
     (property "Reference" "U12"
-      (at 300.48 66.04 0)
+      (at 300.99 66.04 0)
       (effects (font (size 1.27 1.27)))
     )
     (property "Value" "TPS3823-33DBVR"
-      (at 300.48 68.58 0)
+      (at 300.99 68.58 0)
       (effects (font (size 1.27 1.27)))
     )
     (property "Footprint" "Package_TO_SOT_SMD:SOT-23-5"
-      (at 300.48 76.2 0)
+      (at 300.99 76.2 0)
       (effects (font (size 1.27 1.27)) hide)
     )
     (property "Digi-Key_PN" "296-34371-1-ND"
-      (at 300.48 76.2 0)
+      (at 300.99 76.2 0)
       (effects (font (size 1.27 1.27)) hide)
     )
     (property "DNP" "NO"
-      (at 300.48 76.2 0)
+      (at 300.99 76.2 0)
       (effects (font (size 1.27 1.27)) hide)
     )
@@
   (label "5V_RAIL"   (at 170.18 76.2 0)   (effects (font (size 1.27 1.27))) (uuid "nl-5v"))
   (label "3V3_RAIL"  (at 233.68 76.2 0)   (effects (font (size 1.27 1.27))) (uuid "nl-3v3"))
-  (label "WDT_RESET" (at 310.64 73.66 0)  (effects (font (size 1.27 1.27))) (uuid "nl-wdt"))
+  (label "WDT_RESET" (at 311.15 73.66 0)  (effects (font (size 1.27 1.27))) (uuid "nl-wdt"))
   (text "POWER MANAGEMENT BLOCK\n12V → 5V (Buck TPS54302) → 3.3V (LDO AMS1117)\nProtection: TVS + PTC + Schottky\nWatchdog: TPS3823 on all tiers"
     (at 25.4 25.4 0)
