File: kicad/power_management.kicad_sch (KiCad schematic)
At the start: 30 parts, among them J1 PJ-002AH, SW1 RESET, U1 TPS54302DDCR, U2 AMS1117-3.3, U3 TPS3823-33DBVR

Commit message: fix(buck): correct TPS54302 topology — EN UVLO, L1→SW, feedback, output caps
- EN separated from VIN via UVLO divider (R34 100k / R35 18.2k) → ~8V startup,
  protects EN pin (abs-max 6V) from direct 12V
- L1 moved from BOOT net to SW (was on wrong node — buck could not switch to output)
- FB1.2 (ferrite) + input caps C3/C4 tied to filtered VIN; PWR_FLAG on VIN
- Feedback divider completed: R1.1→5V_RAIL, R2 100k... value 24.9k→13.7k for ~4.95V
  (needed ≥4.5V for AMS1117-3.3 LDO input)
- Output cap C6.1→5V_RAIL, LDO output cap C10.1→3V3_RAIL
- Bootstrap C7 preserved between BOOT and SW
- ERC 19→14 (lowered CI threshold accordingly)

Co-Authored-By: Devin AI <158243242+devin-ai-integration[bot]@users.noreply.github.com>
Parts:
- added R34: 100k 1%, Resistor_SMD:R_0402_1005Metric, symbol Device:R
- added R35: 18.2k 1%, Resistor_SMD:R_0402_1005Metric, symbol Device:R
- R2: value 24.9k 1% -> 13.7k 1%; MPN CRCW040224K9FKED -> CRCW040213K7FKED
Connections:
- net 12V_RAIL: no longer C3.1, C4.1, U1.3 (VIN), U1.5 (EN)
- net GND: now also R35.2
- net SW: now reaches C7.1, C7.2, L1.1, U1.2 (SW), U1.6 (BOOT)
- net VIN: now reaches FB1.2
- net VIN: now also C3.1, C4.1, U1.3 (VIN), R34.1
- new net EN_UVLO: R34.2, R35.1, U1.5 (EN)
Changed lines of the file:
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@@
     (uuid "r2-001")
     (property "Reference" "R2" (at 180.34 86.36 0) (effects (font (size 1.27 1.27))))
-    (property "Value" "24.9k 1%" (at 180.34 91.44 0) (effects (font (size 1.27 1.27))))
+    (property "Value" "13.7k 1%" (at 180.34 91.44 0) (effects (font (size 1.27 1.27))))
     (property "Footprint" "Resistor_SMD:R_0402_1005Metric" (at 180.34 88.9 0) (effects (font (size 1.27 1.27)) hide))
-    (property "MPN" "CRCW040224K9FKED" (at 180.34 88.9 0) (effects (font (size 1.27 1.27)) hide))
+    (property "MPN" "CRCW040213K7FKED" (at 180.34 88.9 0) (effects (font (size 1.27 1.27)) hide))
     (pin "1" (uuid "r2-p1")) (pin "2" (uuid "r2-p2"))
     (instances
@@
   )
   (wire
-    (pts (xy 129.54 78.74) (xy 129.54 73.66))
-    (stroke (width 0) (type default))
-  )
-  (wire
     (pts (xy 149.86 76.2) (xy 149.86 67.31))
     (stroke (width 0) (type default))
@@
   )
   (wire
-    (pts (xy 149.86 73.66) (xy 160.02 73.66))
-    (stroke (width 0) (type default))
-  )
-  (wire
-    (pts (xy 160.02 73.66) (xy 160.02 67.31))
-    (stroke (width 0) (type default))
-  )
-  (wire
     (pts (xy 160.02 74.93) (xy 160.02 76.2))
     (stroke (width 0) (type default))
@@
   )
   (wire
-    (pts (xy 175.26 76.2) (xy 175.26 77.47))
-    (stroke (width 0) (type default))
-  )
-  (wire
-    (pts (xy 176.53 76.2) (xy 176.53 81.28))
-    (stroke (width 0) (type default))
-  )
-  (wire
     (pts (xy 184.15 81.28) (xy 184.15 88.9))
     (stroke (width 0) (type default))
@@
   (wire
     (pts (xy 233.68 76.2) (xy 233.68 77.47))
-    (stroke (width 0) (type default))
-  )
-  (wire
-    (pts (xy 241.3 76.2) (xy 241.3 77.47))
     (stroke (width 0) (type default))
   )
@@
     )
   )
-  (label "12V_RAIL" (at 121.92 73.66 0) (effects (font (size 1.27 1.27))))
+  (label "VIN" (at 121.92 73.66 0) (effects (font (size 1.27 1.27))))
   (label "5V_RAIL" (at 208.28 76.2 0) (effects (font (size 1.27 1.27))))
   (label "3V3_RAIL" (at 290.83 68.58 0) (effects (font (size 1.27 1.27))))
@@
   (junction (at 283.21 73.66) (diameter 0) (color 0 0 0 0))
   (junction (at 312.42 68.58) (diameter 0) (color 0 0 0 0))
+  (wire (pts (xy 129.54 73.66) (xy 129.54 71.12)) (stroke (width 0) (type default)))
+  (label "VIN" (at 129.54 71.12 0) (effects (font (size 1.27 1.27)) (justify left bottom)))
+  (wire (pts (xy 105.41 50.8) (xy 113.03 50.8)) (stroke (width 0) (type default)))
+  (label "VIN" (at 109.22 50.8 0) (effects (font (size 1.27 1.27)) (justify left bottom)))
+  (symbol
+    (lib_id "power:PWR_FLAG")
+    (at 113.03 50.8 0)
+    (unit 1)
+    (exclude_from_sim no) (in_bom no) (on_board no)
+    (property "Reference" "#FLG02" (at 113.03 48.26 0) (effects (font (size 1.27 1.27)) hide))
+    (property "Value" "PWR_FLAG" (at 113.03 46.989999999999995 0) (effects (font (size 1.27 1.27))))
+    (pin "1")
+    (instances
+      (project "nebula_qshield"
+        (path "/c6da75fc-541f-4933-b134-f5eb8982a11b/f1fcd624-5e99-46e0-8ec7-0072ddfd5246"
+          (reference "#FLG02") (unit 1)
+        )
+      )
+    )
+  )
+  (wire (pts (xy 129.54 78.74) (xy 129.54 82.55)) (stroke (width 0) (type default)))
+  (label "EN_UVLO" (at 129.54 82.55 0) (effects (font (size 1.27 1.27)) (justify left bottom)))
+  (symbol
+    (lib_id "Device:R")
+    (at 109.22 88.9 0)
+    (unit 1)
+    (exclude_from_sim no) (in_bom yes) (on_board yes)
+    (property "Reference" "R34" (at 111.76 87.63000000000001 0) (effects (font (size 1.27 1.27))))
+    (property "Value" "100k 1%" (at 111.76 90.17 0) (effects (font (size 1.27 1.27))))
+    (property "Footprint" "Resistor_SMD:R_0402_1005Metric" (at 109.22 88.9 0) (effects (font (size 1.27 1.27)) hide))
+    (property "MPN" "CRCW0402100KFKED" (at 109.22 88.9 0) (effects (font (size 1.27 1.27)) hide))
+    (pin "1") (pin "2")
+    (instances
+      (project "nebula_qshield"
+        (path "/c6da75fc-541f-4933-b134-f5eb8982a11b/f1fcd624-5e99-46e0-8ec7-0072ddfd5246"
+          (reference "R34") (unit 1)
+        )
+      )
+    )
+  )
+  (wire (pts (xy 109.22 85.09) (xy 109.22 83.82)) (stroke (width 0) (type default)))
+  (label "VIN" (at 109.22 83.82 0) (effects (font (size 1.27 1.27)) (justify left bottom)))
+  (wire (pts (xy 109.22 92.71) (xy 109.22 96.52)) (stroke (width 0) (type default)))
+  (label "EN_UVLO" (at 109.22 93.98 0) (effects (font (size 1.27 1.27)) (justify left bottom)))
+  (symbol
+    (lib_id "Device:R")
+    (at 109.22 100.33 0)
+    (unit 1)
+    (exclude_from_sim no) (in_bom yes) (on_board yes)
+    (property "Reference" "R35" (at 111.76 99.06 0) (effects (font (size 1.27 1.27))))
+    (property "Value" "18.2k 1%" (at 111.76 101.6 0) (effects (font (size 1.27 1.27))))
+    (property "Footprint" "Resistor_SMD:R_0402_1005Metric" (at 109.22 100.33 0) (effects (font (size 1.27 1.27)) hide))
+    (property "MPN" "CRCW040218K2FKED" (at 109.22 100.33 0) (effects (font (size 1.27 1.27)) hide))
+    (pin "1") (pin "2")
+    (instances
+      (project "nebula_qshield"
+        (path "/c6da75fc-541f-4933-b134-f5eb8982a11b/f1fcd624-5e99-46e0-8ec7-0072ddfd5246"
+          (reference "R35") (unit 1)
+        )
+      )
+    )
+  )
+  (wire (pts (xy 109.22 104.14) (xy 109.22 105.41)) (stroke (width 0) (type default)))
+  (symbol
+    (lib_id "power:GND")
+    (at 109.22 105.41 0)
+    (unit 1)
+    (exclude_from_sim no) (in_bom no) (on_board no)
+    (property "Reference" "#PWR21" (at 109.22 107.95 0) (effects (font (size 1.27 1.27)) hide))
+    (property "Value" "GND" (at 109.22 106.67999999999999 0) (effects (font (size 1.27 1.27)) hide))
+    (pin "1")
+    (instances
+      (project "nebula_qshield"
+        (path "/c6da75fc-541f-4933-b134-f5eb8982a11b/f1fcd624-5e99-46e0-8ec7-0072ddfd5246"
+          (reference "#PWR21") (unit 1)
+        )
+      )
+    )
+  )
+  (label "SW" (at 149.86 67.31 0) (effects (font (size 1.27 1.27)) (justify left bottom)))
+  (wire (pts (xy 160.02 67.31) (xy 163.83 67.31)) (stroke (width 0) (type default)))
+  (label "SW" (at 163.83 67.31 0) (effects (font (size 1.27 1.27)) (justify left bottom)))
+  (wire (pts (xy 176.53 81.28) (xy 176.53 76.2)) (stroke (width 0) (type default)))
+  (label "5V_RAIL" (at 176.53 78.74 0) (effects (font (size 1.27 1.27)) (justify left bottom)))
+  (wire (pts (xy 175.26 77.47) (xy 175.26 76.2)) (stroke (width 0) (type default)))
+  (label "5V_RAIL" (at 175.26 77.47 0) (effects (font (size 1.27 1.27)) (justify left bottom)))
+  (wire (pts (xy 241.3 77.47) (xy 245.11 77.47)) (stroke (width 0) (type default)))
+  (label "3V3_RAIL" (at 245.11 77.47 0) (effects (font (size 1.27 1.27)) (justify left bottom)))
 )

Commit message: fix(erc): clean remaining ERC violations in hierarchical schematics
- Reconnect 5V_RAIL and 3V3_RAIL hierarchical labels in power_management.
- Move MCU_WDI hierarchical label to U3 WDI and add R3 pull-up wiring.
- Add PWR_FLAG sources for GND (power_management) and PGND (actuator_drivers).
- Add 5V_RAIL PWR_FLAG in power_management.
- Remove redundant PWR_FLAGS #FLG40 and #FLG41 from analog_acquisition.
- Place no_connect markers on unused MAX485 U15 left-side pins.
- Change HX711 AVDD pin type from power_out to power_in (library and digital sheet).
- Change Arduino shield header 5V/3V3 pins from power_out to passive.
- Achieve zero ERC violations in kicad-cli sch erc.

Co-Authored-By: Devin AI <158243242+devin-ai-integration[bot]@users.noreply.github.com>
Changed lines of the file:
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@@
   (hierarchical_label "3V3_RAIL"   (shape output)   (at 248.92 76.2 0)  (effects (font (size 1.27 1.27))) (uuid "hl-3v3"))
   (hierarchical_label "GND"        (shape bidirectional) (at 25.4 58.42 270)   (effects (font (size 1.27 1.27))) (uuid "hl-gnd"))
-  (hierarchical_label "MCU_WDI"    (shape input)    (at 279.4 73.66 180) (effects (font (size 1.27 1.27))) (uuid "hl-wdi"))
+  (hierarchical_label "MCU_WDI"    (shape input)    (at 293.37 73.66 180) (effects (font (size 1.27 1.27))) (uuid "hl-wdi"))
   (hierarchical_label "MCU_NRST"   (shape output)   (at 320.04 73.66 0) (effects (font (size 1.27 1.27))) (uuid "hl-nrst"))
   (label "VIN_12V"   (at 30.48 50.8 0)    (effects (font (size 1.27 1.27))) (uuid "nl-vin"))
@@
   )
   (wire
+    (pts (xy 33.02 58.42) (xy 35.56 58.42))
+    (stroke (width 0) (type default))
+  )
+  (wire
+    (pts (xy 35.56 58.42) (xy 40.64 58.42))
+    (stroke (width 0) (type default))
+  )
+  (symbol
+    (lib_id "power:PWR_FLAG")
+    (at 35.56 58.42 0)
+    (unit 1)
+    (exclude_from_sim no)
+    (in_bom no)
+    (on_board no)
+    (property "Reference" "#FLG04"
+      (at 35.56 55.88 0)
+      (effects (font (size 1.27 1.27)) hide)
+    )
+    (property "Value" "PWR_FLAG"
+      (at 35.56 54.61 0)
+      (effects (font (size 1.27 1.27)) hide)
+    )
+    (pin "1"
+    )
+    (instances
+      (project "nebula_qshield"
+        (path "/c6da75fc-541f-4933-b134-f5eb8982a11b/f1fcd624-5e99-46e0-8ec7-0072ddfd5246"
+          (reference "#FLG04") (unit 1)
+        )
+      )
+    )
+  )
+  (wire
     (pts (xy 121.92 73.66) (xy 129.54 73.66))
     (stroke (width 0) (type default))
@@
   )
   (wire
+    (pts (xy 187.96 76.2) (xy 208.28 76.2))
+    (stroke (width 0) (type default))
+  )
+  (wire
     (pts (xy 170.18 76.2) (xy 170.18 77.47))
     (stroke (width 0) (type default))
@@
     (stroke (width 0) (type default))
   )
+  (symbol
+    (lib_id "power:PWR_FLAG")
+    (at 208.28 77.47 0)
+    (unit 1)
+    (exclude_from_sim no)
+    (in_bom no)
+    (on_board no)
+    (property "Reference" "#FLG05"
+      (at 208.28 76.2 0)
+      (effects (font (size 1.27 1.27)) hide)
+    )
+    (property "Value" "PWR_FLAG"
+      (at 208.28 75.94 0)
+      (effects (font (size 1.27 1.27)) hide)
+    )
+    (pin "1"
+    )
+    (instances
+      (project "nebula_qshield"
+        (path "/c6da75fc-541f-4933-b134-f5eb8982a11b/f1fcd624-5e99-46e0-8ec7-0072ddfd5246"
+          (reference "#FLG05") (unit 1)
+        )
+      )
+    )
+  )
   (wire
     (pts (xy 228.6 76.2) (xy 248.92 76.2))
@@
   )
   (wire
+    (pts (xy 248.92 76.2) (xy 251.46 76.2))
+    (stroke (width 0) (type default))
+  )
+  (label "3V3_RAIL" (at 251.46 76.2 0) (effects (font (size 1.27 1.27))))
+  (wire
     (pts (xy 233.68 76.2) (xy 233.68 77.47))
     (stroke (width 0) (type default))
@@
   )
   (wire
-    (pts (xy 279.4 73.66) (xy 290.83 73.66))
-    (stroke (width 0) (type default))
-  )
+    (pts (xy 293.37 73.66) (xy 290.83 73.66))
+    (stroke (width 0) (type default))
+  )
+  (wire
+    (pts (xy 283.21 73.66) (xy 290.83 73.66))
+    (stroke (width 0) (type default))
+  )

Commit message: feat(sch,pcb,docs): redefine tiers Essential/Insight/Signature and sync DNP
- Tier mapping:
  - Essential: GPS, RTC/timestamp, temperature, pH, ORP
  - Insight: Essential + CO2 pressure (A4), DO (A5), HX711 load cell,
    chiller, recirculation motor, gas solenoid (single gas via K1/J18)
  - Signature: Insight + Hamilton TCD + ACD via RS485 bridge
- Humidity channel (J7/D8/R17/R18/C23) and PWM gas valve (U20/Q5/D14/R28/C27/J22)
  marked DNP in all tiers.
- Update DNP properties in kicad/analog_acquisition.kicad_sch,
  kicad/digital_i2c.kicad_sch, kicad/actuator_drivers.kicad_sch,
  kicad/power_management.kicad_sch using kicad/tier_dnp_mapping.json.
- Update sheet comments and root text block.
- Update docs/04_BOM_PRODUCTION.md section 11, docs/INSIGHT_FABRICATION_ROADMAP.md,
  and docs/DOCUMENTATION_UPDATE_AUDIT.md.
- Add helper tools: build_tier_map.py, apply_tier_dnp4.py, update_tier_comments.py,
  list_actual_components.py, tier_counts.py, validate_sch.py, count_parens.py.
- Sync current PCB state (component positions/nets) to match corrected netlist.

Validation:
- kicad-cli sch erc --severity-all: 0 violaciones
- kicad-cli pcb drc --severity-error: 0 violaciones, 332 unconnected items
- compare_pcb_to_netlist.py: 0 parity problems

Co-Authored-By: Devin AI <158243242+devin-ai-integration[bot]@users.noreply.github.com>
Parts:
- C1, C10, C11, C2, C3, C4, C5, C6, C7, C8, C9, D1, D2, F1, FB1, J1, L1, LED1, LED2, LED3, R1, R2, R3, R34, R35, R4, R5, R6, SW1, U1, U2: DNP (none) -> NO
